File: D1MSERVO.sch (EAGLE design)
At the start: 57 parts, among them IC1 PCA9685

Commit message: Changed I2C pins
Connections:
- net D4: now also SJ7.1
- net D5: now also SJ8.1
- net D6: no longer SJ7.1
- net D7: no longer SJ8.1
Changed lines of the file:
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@@
 <label x="27.94" y="154.94" size="1.778" layer="95"/>
+</segment>
+<segment>
+<pinref part="SJ8" gate="G$1" pin="1"/>
+<wire x1="33.02" y1="91.44" x2="27.94" y2="91.44" width="0.1524" layer="91"/>
+<label x="30.48" y="91.44" size="1.778" layer="95"/>
 </segment>
 </net>
@@
 <pinref part="H1" gate="G$1" pin="5"/>
 </segment>
-<segment>
-<pinref part="SJ7" gate="G$1" pin="1"/>
-<wire x1="38.1" y1="99.06" x2="27.94" y2="99.06" width="0.1524" layer="91"/>
-<label x="30.48" y="99.06" size="1.778" layer="95"/>
-</segment>
 </net>
 <net name="D7" class="0">
@@
 <wire x1="26.67" y1="149.86" x2="38.1" y2="149.86" width="0.1524" layer="91"/>
 <label x="27.94" y="149.86" size="1.778" layer="95"/>
-</segment>
-<segment>
-<pinref part="SJ8" gate="G$1" pin="1"/>
-<wire x1="33.02" y1="91.44" x2="27.94" y2="91.44" width="0.1524" layer="91"/>
-<label x="30.48" y="91.44" size="1.778" layer="95"/>
 </segment>
 </net>
@@
 <label x="49.53" y="149.86" size="1.778" layer="95"/>
 </segment>
+<segment>
+<pinref part="SJ7" gate="G$1" pin="1"/>
+<wire x1="38.1" y1="99.06" x2="27.94" y2="99.06" width="0.1524" layer="91"/>
+<label x="30.48" y="99.06" size="1.778" layer="95"/>
+</segment>
 </net>

Commit message: Changed I2C pins (again) to match ESP12E like on the D1 Mini and D1 R2
Connections:
- net D1: now also SJ8.1
- net D2: now also SJ7.1
- net D4: no longer SJ7.1
- net D5: no longer SJ8.1
Changed lines of the file:
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@@
 <label x="49.53" y="157.48" size="1.778" layer="95"/>
+</segment>
+<segment>
+<pinref part="SJ8" gate="G$1" pin="1"/>
+<wire x1="33.02" y1="91.44" x2="27.94" y2="91.44" width="0.1524" layer="91"/>
+<label x="30.48" y="91.44" size="1.778" layer="95"/>
 </segment>
 </net>
@@
 <label x="49.53" y="154.94" size="1.778" layer="95"/>
 </segment>
+<segment>
+<pinref part="SJ7" gate="G$1" pin="1"/>
+<wire x1="38.1" y1="99.06" x2="27.94" y2="99.06" width="0.1524" layer="91"/>
+<label x="30.48" y="99.06" size="1.778" layer="95"/>
+</segment>
 </net>
 <net name="D5" class="0">
@@
 <wire x1="26.67" y1="154.94" x2="38.1" y2="154.94" width="0.1524" layer="91"/>
 <label x="27.94" y="154.94" size="1.778" layer="95"/>
-</segment>
-<segment>
-<pinref part="SJ8" gate="G$1" pin="1"/>
-<wire x1="33.02" y1="91.44" x2="27.94" y2="91.44" width="0.1524" layer="91"/>
-<label x="30.48" y="91.44" size="1.778" layer="95"/>
 </segment>
 </net>
@@
 <label x="49.53" y="149.86" size="1.778" layer="95"/>
 </segment>
-<segment>
-<pinref part="SJ7" gate="G$1" pin="1"/>
-<wire x1="38.1" y1="99.06" x2="27.94" y2="99.06" width="0.1524" layer="91"/>
-<label x="30.48" y="99.06" size="1.778" layer="95"/>
-</segment>
 </net>
